File: boards/imx6ull-devboard/hardware/layouts/default/default.kicad_pcb (KiCad board)
At the start: 2 copper layers, 181 parts, among them Q1 Vgs ℝ+V

Commit message: DDR3 module written + datasheet-verified, build blocker documented
DDR3 subsystem (Nanya NT5CC128M16JR-EK, 96-ball TFBGA, 256 MB):
- src/ddr3.ato: 89-line wrapper, full pin mapping verified against datasheet
  pages 4-7. DQSL pair fix (was swapped in auto-gen). 12× 100nF decoupling +
  2× 10µF bulk + 240Ω ZQ resistor. VREFCA + VREFDQ both via bus.vref.
- src/parts/Nanya_Tech_NT5CC128M16JR_EK/: atomic part with fixes:
    * 6 NC pads added (J1, J9, L1, L9, M7, T7)
    * Address signals prefixed (DDR_A0, DDR_A4, etc.) to avoid collision
      with i.MX 6ULL BGA pad coordinates
- mpu.ato: added vref field to DDR3Bus interface, wired DRAM_VREF to it
- docs/subsystems/ddr3.md: full design doc + investigation log

KNOWN BLOCKER documented in CLAUDE.md and ddr3.md:
  ato build crashes with "min() iterable argument is empty" during PCB-write
  stage as soon as the DDR3 chip is instantiated, even with zero connections.
  atopile log DB shows MPU pad-coordinate-named nets being renamed when DDR3
  enters the design; something in the rename path leaves an empty pad list.
  Schematic side IS correct — only the build-time PCB write fails.

CLAUDE.md updated with full project state, known atopile gotchas (6 of them
hit in this project), DDR3 debug pack with diagnostic clues + faebryk source
paths + next-step hypotheses, and quick command reference.

DDR3 instantiation commented out in main.ato so the rest of the board still
builds successfully (58-line BOM + KiCad PCB).

Co-Authored-By: Claude Opus 4.7 (1M context) <noreply@anthropic.com>
Connections:
- net mpu-ddr3-line renamed DRAM_ADDR00
- net mpu-ddr3-line-1 renamed DRAM_ADDR10
- net mpu-ddr3-line-10 renamed DRAM_ADDR04
- net mpu-ddr3-line-11 renamed DRAM_ADDR05
- net mpu-ddr3-line-12 renamed DRAM_ADDR06
- net mpu-ddr3-line-13 renamed DRAM_ADDR07
- net mpu-ddr3-line-14 renamed DRAM_ADDR08
- net mpu-ddr3-line-15 renamed DRAM_ADDR09
- net mpu-ddr3-line-16 renamed DRAM_SDBA0
- net mpu-ddr3-line-17 renamed DRAM_SDBA1
- net mpu-ddr3-line-18 renamed DRAM_SDBA2
- net mpu-ddr3-line-19 renamed DRAM_DATA00
- net mpu-ddr3-line-2 renamed DRAM_ADDR11
- net mpu-ddr3-line-20 renamed DRAM_DATA10
- net mpu-ddr3-line-21 renamed DRAM_DATA11
- net mpu-ddr3-line-22 renamed DRAM_DATA12
- net mpu-ddr3-line-23 renamed DRAM_DATA13
- net mpu-ddr3-line-24 renamed DRAM_DATA14
- net mpu-ddr3-line-25 renamed DRAM_DATA15
- net mpu-ddr3-line-26 renamed DRAM_DATA01
- net mpu-ddr3-line-27 renamed DRAM_DATA02
- net mpu-ddr3-line-28 renamed DRAM_DATA03
- net mpu-ddr3-line-29 renamed DRAM_DATA04
- net mpu-ddr3-line-3 renamed DRAM_ADDR12
- net mpu-ddr3-line-30 renamed DRAM_DATA05
- net mpu-ddr3-line-31 renamed DRAM_DATA06
- net mpu-ddr3-line-32 renamed DRAM_DATA07
- net mpu-ddr3-line-33 renamed DRAM_DATA08
- net mpu-ddr3-line-34 renamed DRAM_DATA09
- net mpu-ddr3-line-35 renamed DRAM_DQM0
- net mpu-ddr3-line-36 renamed DRAM_DQM1
- net mpu-ddr3-line-37 renamed DRAM_ODT0
- net mpu-ddr3-line-38 renamed DRAM_SDCKE0
- net mpu-ddr3-line-4 renamed DRAM_ADDR13
- net mpu-ddr3-line-5 renamed DRAM_ADDR14
- net mpu-ddr3-line-6 renamed DRAM_ADDR15
- net mpu-ddr3-line-7 renamed DRAM_ADDR01
- net mpu-ddr3-line-8 renamed DRAM_ADDR02
- net mpu-ddr3-line-9 renamed DRAM_ADDR03
Changed lines of the file:
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@@
 	(net 187 "CSI_HSYNC")
 	(net 188 "CSI_MCLK")
-	(net 189 "mpu-ddr3-line-5")
+	(net 189 "DRAM_ADDR14")
 	(net 190 "UART4_RX_DATA")
 	(net 191 "UART4_TX_DATA")
-	(net 192 "mpu-ddr3-line-12")
-	(net 193 "mpu-ddr3-line-17")
+	(net 192 "DRAM_ADDR06")
+	(net 193 "DRAM_SDBA1")
 	(net 194 "power_1v4_arm-hv")
 	(net 195 "UART2_RTS_B")
@@
 	(net 197 "UART3_RX_DATA")
 	(net 198 "UART3_TX_DATA")
-	(net 199 "mpu-ddr3-line-7")
-	(net 200 "mpu-ddr3-line-4")
-	(net 201 "mpu-ddr3-line-13")
+	(net 199 "DRAM_ADDR01")
+	(net 200 "DRAM_ADDR13")
+	(net 201 "DRAM_ADDR07")
 	(net 202 "DRAM_CS1_B")
 	(net 203 "VDD_SOC_IN")
@@
 	(net 208 "DRAM_CAS_B")
 	(net 209 "DRAM_SDCKE1")
-	(net 210 "mpu-ddr3-line-14")
-	(net 211 "mpu-ddr3-line-8")
+	(net 210 "DRAM_ADDR08")
+	(net 211 "DRAM_ADDR02")
 	(net 212 "usb_otg1_id-line")
 	(net 213 "UART1_TX_DATA")
@@
 	(net 215 "UART1_RX_DATA")
 	(net 216 "GPIO1_IO06")
-	(net 217 "mpu-ddr3-line-18")
-	(net 218 "mpu-ddr3-line-2")
-	(net 219 "mpu-ddr3-line-10")
-	(net 220 "mpu-ddr3-line-6")
-	(net 221 "mpu-ddr3-line-11")
+	(net 217 "DRAM_SDBA2")
+	(net 218 "DRAM_ADDR11")
+	(net 219 "DRAM_ADDR04")
+	(net 220 "DRAM_ADDR15")
+	(net 221 "DRAM_ADDR05")
 	(net 222 "GPIO1_IO01")
 	(net 223 "GPIO1_IO07")
 	(net 224 "line")
-	(net 225 "mpu-ddr3-line-15")
-	(net 226 "mpu-ddr3-line-3")
-	(net 227 "mpu-ddr3-line")
-	(net 228 "mpu-ddr3-line-16")
+	(net 225 "DRAM_ADDR09")
+	(net 226 "DRAM_ADDR12")
+	(net 227 "DRAM_ADDR00")
+	(net 228 "DRAM_SDBA0")
 	(net 229 "M12")
 	(net 230 "GPIO1_IO04")
 	(net 231 "GPIO1_IO05")
-	(net 232 "mpu-ddr3-line-9")
-	(net 233 "mpu-ddr3-line-38")
-	(net 234 "mpu-ddr3-line-1")
+	(net 232 "DRAM_ADDR03")
+	(net 233 "DRAM_SDCKE0")
+	(net 234 "DRAM_ADDR10")
 	(net 235 "DRAM_RAS_B")
-	(net 236 "mpu-ddr3-line-37")
+	(net 236 "DRAM_ODT0")
 	(net 237 "N10")
 	(net 238 "N11")
@@
 	(net 253 "CCM_CLK1_P")
 	(net 254 "DRAM_SDCLK0_N")
-	(net 255 "mpu-ddr3-line-23")
-	(net 256 "mpu-ddr3-line-22")
+	(net 255 "DRAM_DATA13")
+	(net 256 "DRAM_DATA12")
 	(net 257 "DRAM_SDQS0_P")
 	(net 258 "DRAM_SDQS0_N")
 	(net 259 "SNVS_TAMPER4")
-	(net 260 "mpu-ddr3-line-25")
+	(net 260 "DRAM_DATA15")
 	(net 261 "R10")
 	(net 262 "GPANAIO")
 	(net 263 "cap_ud_high-power-hv")
-	(net 264 "mpu-ddr3-line-24")
+	(net 264 "DRAM_DATA14")
 	(net 265 "R6")
 	(net 266 "R9")
@@
 	(net 273 "cap_xtal_b-power-hv")
 	(net 274 "DRAM_SDQS1_N")
-	(net 275 "mpu-ddr3-line-36")
-	(net 276 "mpu-ddr3-line-19")
-	(net 277 "mpu-ddr3-line-31")
-	(net 278 "mpu-ddr3-line-27")
-	(net 279 "mpu-ddr3-line-35")
-	(net 280 "mpu-ddr3-line-30")
+	(net 275 "DRAM_DQM1")
+	(net 276 "DRAM_DATA00")
+	(net 277 "DRAM_DATA06")
+	(net 278 "DRAM_DATA02")
+	(net 279 "DRAM_DQM0")
+	(net 280 "DRAM_DATA05")
 	(net 281 "SNVS_PMIC_ON_REQ")
 	(net 282 "JTAG_MOD")
@@
 	(net 52 "UART3_RTS_B")
 	(net 55 "DRAM_RESET")
-	(net 64 "mpu-ddr3-line-21")
+	(net 64 "DRAM_DATA11")
 	(net 65 "RTC_XTALO")
 	(net 66 "USB_OTG2_VBUS")
@@
 	(net 74 "USB_OTG1_DP_P")
 	(net 75 "USB_OTG1_CHD_B")
-	(net 76 "mpu-ddr3-line-33")
-	(net 77 "mpu-ddr3-line-34")
-	(net 78 "mpu-ddr3-line-32")
-	(net 79 "mpu-ddr3-line-20")
-	(net 80 "mpu-ddr3-line-26")
-	(net 94 "mpu-ddr3-line-28")
-	(net 95 "mpu-ddr3-line-29")
+	(net 76 "DRAM_DATA08")
+	(net 77 "DRAM_DATA09")
+	(net 78 "DRAM_DATA07")
+	(net 79 "DRAM_DATA10")
+	(net 80 "DRAM_DATA01")
+	(net 94 "DRAM_DATA03")
+	(net 95 "DRAM_DATA04")
 	(net 96 "CCM_PMIC_STBY_REQ")
 	(net 97 "CSI_DATA03")
@@
 			(size 0.32 0.32)
 			(layers "F.Cu" "F.Paste" "F.Mask")
-			(net 189 "mpu-ddr3-line-5")
+			(net 189 "DRAM_ADDR14")
 		)
 		(pad "H1" smd circle
@@
 			(size 0.32 0.32)
 			(layers "F.Cu" "F.Paste" "F.Mask")
-			(net 193 "mpu-ddr3-line-17")
+			(net 193 "DRAM_SDBA1")
 		)
 		(pad "J1" smd circle
@@
 			(size 0.32 0.32)
 			(layers "F.Cu" "F.Paste" "F.Mask")
-			(net 211 "mpu-ddr3-line-8")
+			(net 211 "DRAM_ADDR02")
 		)
 		(pad "L1" smd circle
@@
 			(size 0.32 0.32)
 			(layers "F.Cu" "F.Paste" "F.Mask")
-			(net 221 "mpu-ddr3-line-11")
+			(net 221 "DRAM_ADDR05")
 		)
 		(pad "M1" smd circle
@@
 			(size 0.32 0.32)
 			(layers "F.Cu" "F.Paste" "F.Mask")
-			(net 228 "mpu-ddr3-line-16")
+			(net 228 "DRAM_SDBA0")
 		)
 		(pad "N1" smd circle
@@
 			(size 0.32 0.32)
 			(layers "F.Cu" "F.Paste" "F.Mask")
-			(net 236 "mpu-ddr3-line-37")
+			(net 236 "DRAM_ODT0")
 		)
 		(pad "P1" smd circle
@@
 			(size 0.32 0.32)
 			(layers "F.Cu" "F.Paste" "F.Mask")
-			(net 260 "mpu-ddr3-line-25")
+			(net 260 "DRAM_DATA15")
 		)
 		(pad "T1" smd circle
@@
 			(size 0.32 0.32)
 			(layers "F.Cu" "F.Paste" "F.Mask")
-			(net 192 "mpu-ddr3-line-12")
+			(net 192 "DRAM_ADDR06")
 		)
 		(pad "H2" smd circle
@@
 			(size 0.32 0.32)
 			(layers "F.Cu" "F.Paste" "F.Mask")
-			(net 199 "mpu-ddr3-line-7")
+			(net 199 "DRAM_ADDR01")
 		)
 		(pad "J2" smd circle
@@
 			(size 0.32 0.32)
 			(layers "F.Cu" "F.Paste" "F.Mask")
-			(net 217 "mpu-ddr3-line-18")
+			(net 217 "DRAM_SDBA2")
 		)
 		(pad "L2" smd circle
@@
 			(size 0.32 0.32)
 			(layers "F.Cu" "F.Paste" "F.Mask")
-			(net 225 "mpu-ddr3-line-15")
+			(net 225 "DRAM_ADDR09")
 		)
 		(pad "M2" smd circle
@@
 			(size 0.32 0.32)
 			(layers "F.Cu" "F.Paste" "F.Mask")
-			(net 232 "mpu-ddr3-line-9")
+			(net 232 "DRAM_ADDR03")
 		)
 		(pad "N2" smd circle
@@
 			(size 0.32 0.32)
 			(layers "F.Cu" "F.Paste" "F.Mask")
-			(net 264 "mpu-ddr3-line-24")
+			(net 264 "DRAM_DATA14")
 		)
 		(pad "T2" smd circle
@@
 			(size 0.32 0.32)
 			(layers "F.Cu" "F.Paste" "F.Mask")
-			(net 76 "mpu-ddr3-line-33")
+			(net 76 "DRAM_DATA08")
 		)
 		(pad "A3" smd circle
@@
 			(size 0.32 0.32)
 			(layers "F.Cu" "F.Paste" "F.Mask")
-			(net 200 "mpu-ddr3-line-4")
+			(net 200 "DRAM_ADDR13")
 		)
 		(pad "J3" smd circle
@@
 			(size 0.32 0.32)
 			(layers "F.Cu" "F.Paste" "F.Mask")
-			(net 218 "mpu-ddr3-line-2")
+			(net 218 "DRAM_ADDR11")
 		)
 		(pad "L3" smd circle
@@
 			(size 0.32 0.32)
 			(layers "F.Cu" "F.Paste" "F.Mask")
-			(net 233 "mpu-ddr3-line-38")
+			(net 233 "DRAM_SDCKE0")
 		)
 		(pad "N3" smd circle
@@
 			(size 0.32 0.32)
 			(layers "F.Cu" "F.Paste" "F.Mask")
-			(net 255 "mpu-ddr3-line-23")
+			(net 255 "DRAM_DATA13")
 		)
 		(pad "R3" smd circle
@@
 			(size 0.32 0.32)
 			(layers "F.Cu" "F.Paste" "F.Mask")
-			(net 275 "mpu-ddr3-line-36")
+			(net 275 "DRAM_DQM1")
 		)
 		(pad "U3" smd circle
@@
 			(size 0.32 0.32)
 			(layers "F.Cu" "F.Paste" "F.Mask")
-			(net 77 "mpu-ddr3-line-34")
+			(net 77 "DRAM_DATA09")
 		)
 		(pad "A4" smd circle
@@
 			(size 0.32 0.32)
 			(layers "F.Cu" "F.Paste" "F.Mask")
-			(net 201 "mpu-ddr3-line-13")
+			(net 201 "DRAM_ADDR07")
 		)
 		(pad "J4" smd circle
@@
 			(size 0.32 0.32)
 			(layers "F.Cu" "F.Paste" "F.Mask")
-			(net 210 "mpu-ddr3-line-14")
+			(net 210 "DRAM_ADDR08")
 		)
 		(pad "K4" smd circle
@@
 			(size 0.32 0.32)
 			(layers "F.Cu" "F.Paste" "F.Mask")
-			(net 219 "mpu-ddr3-line-10")
+			(net 219 "DRAM_ADDR04")
 		)
 		(pad "L4" smd circle
@@
 			(size 0.32 0.32)
 			(layers "F.Cu" "F.Paste" "F.Mask")
-			(net 226 "mpu-ddr3-line-3")
+			(net 226 "DRAM_ADDR12")
 		)
 		(pad "M4" smd circle
@@
 			(size 0.32 0.32)
 			(layers "F.Cu" "F.Paste" "F.Mask")
-			(net 234 "mpu-ddr3-line-1")
+			(net 234 "DRAM_ADDR10")
 		)
 		(pad "N4" smd circle
@@
 			(size 0.32 0.32)
 			(layers "F.Cu" "F.Paste" "F.Mask")
-			(net 64 "mpu-ddr3-line-21")
+			(net 64 "DRAM_DATA11")
 		)
 		(pad "T4" smd circle
@@
 			(size 0.32 0.32)
 			(layers "F.Cu" "F.Paste" "F.Mask")
-			(net 276 "mpu-ddr3-line-19")
+			(net 276 "DRAM_DATA00")
 		)
 		(pad "U4" smd circle
@@
 			(size 0.32 0.32)
 			(layers "F.Cu" "F.Paste" "F.Mask")
-			(net 78 "mpu-ddr3-line-32")
+			(net 78 "DRAM_DATA07")
 		)
 		(pad "A5" smd circle
@@
 			(size 0.32 0.32)
 			(layers "F.Cu" "F.Paste" "F.Mask")
-			(net 220 "mpu-ddr3-line-6")
+			(net 220 "DRAM_ADDR15")
 		)
 		(pad "L5" smd circle
@@
 			(size 0.32 0.32)
 			(layers "F.Cu" "F.Paste" "F.Mask")
-			(net 227 "mpu-ddr3-line")
+			(net 227 "DRAM_ADDR00")
 		)
 		(pad "M5" smd circle
@@
 			(size 0.32 0.32)
 			(layers "F.Cu" "F.Paste" "F.Mask")
-			(net 256 "mpu-ddr3-line-22")
+			(net 256 "DRAM_DATA12")
 		)
 		(pad "R5" smd circle
@@
 			(size 0.32 0.32)
 			(layers "F.Cu" "F.Paste" "F.Mask")
-			(net 277 "mpu-ddr3-line-31")
+			(net 277 "DRAM_DATA06")
 		)
 		(pad "U5" smd circle
@@
 			(size 0.32 0.32)
 			(layers "F.Cu" "F.Paste" "F.Mask")
-			(net 79 "mpu-ddr3-line-20")
+			(net 79 "DRAM_DATA10")
 		)
 		(pad "A6" smd circle
@@
 			(size 0.32 0.32)
 			(layers "F.Cu" "F.Paste" "F.Mask")
-			(net 278 "mpu-ddr3-line-27")
+			(net 278 "DRAM_DATA02")
 		)
 		(pad "U6" smd circle
@@
 			(size 0.32 0.32)
 			(layers "F.Cu" "F.Paste" "F.Mask")
-			(net 80 "mpu-ddr3-line-26")
+			(net 80 "DRAM_DATA01")
 		)
 		(pad "A7" smd circle
@@
 			(size 0.32 0.32)
 			(layers "F.Cu" "F.Paste" "F.Mask")
-			(net 279 "mpu-ddr3-line-35")
+			(net 279 "DRAM_DQM0")
 		)
 		(pad "U7" smd circle
@@
 			(size 0.32 0.32)
 			(layers "F.Cu" "F.Paste" "F.Mask")
-			(net 94 "mpu-ddr3-line-28")
+			(net 94 "DRAM_DATA03")
 		)
 		(pad "A8" smd circle
@@
 			(size 0.32 0.32)
 			(layers "F.Cu" "F.Paste" "F.Mask")
-			(net 280 "mpu-ddr3-line-30")
+			(net 280 "DRAM_DATA05")
 		)
 		(pad "U8" smd circle
@@
 			(size 0.32 0.32)
 			(layers "F.Cu" "F.Paste" "F.Mask")
-			(net 95 "mpu-ddr3-line-29")
+			(net 95 "DRAM_DATA04")
 		)
 		(pad "A9" smd circle

Commit message: Wire crystals, USB-C OTG, RJ45 magjack, and I²C RTC — 4 schematic-side blockers fixed
- Crystals (#1): real 24 MHz YXC X322524MOB4SI (C70590) + 2× Epson FC-135
  (C32346, one for SoC RTC and one for the new external RTC). Kills the prior
  "no footprint for xtal_main / xtal_rtc" warnings — board now has a clock.

- USB-C OTG #2 (#2): new src/usb_otg.ato wrapping atopile/usb-connectors
  (5.1k CC pulldowns → UFP/device, 1A fuse, USBLC6 ESD). Fixed the broken
  20k/30k VBUS divider in mpu.ato that pulled VBUS to 3V at the chip pin —
  i.MX VBUS_VALID threshold is ~4.4V, so OTG would never have enabled.
  Replaced with a 100Ω series resistor per NXP AN12028. ID pin pulled HIGH
  inside the MPU module via 100k → device-mode default.

- Ethernet magjack (#3): HR911105A (C12074) with Bob Smith network (2× 75Ω
  center taps + 1nF/2kV X1Y1 to chassis GND), 1MΩ static drain, and 2× 330Ω
  LED resistors driving link/speed bezel LEDs from PHY active-low cathodes.
  Fixed EasyEDA pin-label bug (used cable-side RJ pin numbering instead of
  PCB-side pad numbering — corrected to canonical Hanrun datasheet pinout).

- External I²C RTC (bonus): NXP PCF8563T (C7440) with own 32.768 kHz xtal,
  battery-backed via VDD_SNVS (coin-cell-OR'd in PowerTree). Fixed EasyEDA
  bug claiming OSCI=pin 9 on a SOIC-8 (corrected to pin 1). Added new I²C1
  interface to MPU on UART4_TX/RX pads (ALT2 confirmed against
  imx6ul-pinfunc.h via WebFetch). Bus is multi-drop ready for future PMIC.

Build state: 11/11 subsystems shipping, 66-line BOM, clean ato build.

Co-Authored-By: Claude Opus 4.7 (1M context) <noreply@anthropic.com>
Parts:
- added C100: 100nF ±10%, Samsung_Electro_Mechanics_CL05B104KO5NNNC:C0402, F.Cu at (10.0, -54.0)
- added C101: 100nF ±10%, Samsung_Electro_Mechanics_CL05B104KO5NNNC:C0402, F.Cu at (10.0, -60.0)
- added C102: 100nF ±10%, Samsung_Electro_Mechanics_CL05B104KO5NNNC:C0402, F.Cu at (10.0, -66.0)
- added C103: 100nF ±10%, Samsung_Electro_Mechanics_CL05B104KO5NNNC:C0402, F.Cu at (10.0, -72.0)
- added C104: 100nF ±10%, Samsung_Electro_Mechanics_CL05B104KO5NNNC:C0402, F.Cu at (10.0, -78.0)
- added C105: 100nF ±10%, Samsung_Electro_Mechanics_CL05B104KO5NNNC:C0402, F.Cu at (10.0, -18.0)
- added C106: 100nF ±10%, Samsung_Electro_Mechanics_CL05B104KO5NNNC:C0402, F.Cu at (10.0, -24.0)
- added C107: 100nF ±10%, Samsung_Electro_Mechanics_CL05B104KO5NNNC:C0402, F.Cu at (2.25, -6.50)
- added C108: 100nF ±10%, Samsung_Electro_Mechanics_CL05B104KO5NNNC:C0402, F.Cu at (20.0, 0.00)
- added C109: 1nF ±10%, Samsung_Electro_Mechanics_CL21B102KBCNNNC:C0805, F.Cu at (10.0, 0.00)
- added C93: 10µF ±10%, Samsung_Electro_Mechanics_CL21A106KAYNNNE:C0805, F.Cu at (10.0, 0.00)
- added C94: 10µF ±10%, Samsung_Electro_Mechanics_CL21A106KAYNNNE:C0805, F.Cu at (10.0, -6.00)
- added C95: 100nF ±10%, Samsung_Electro_Mechanics_CL05B104KO5NNNC:C0402, F.Cu at (10.0, -12.0)
- added C96: 100nF ±10%, Samsung_Electro_Mechanics_CL05B104KO5NNNC:C0402, F.Cu at (10.0, -30.0)
- added C97: 100nF ±10%, Samsung_Electro_Mechanics_CL05B104KO5NNNC:C0402, F.Cu at (10.0, -36.0)
- added C98: 100nF ±10%, Samsung_Electro_Mechanics_CL05B104KO5NNNC:C0402, F.Cu at (10.0, -42.0)
- added C99: 100nF ±10%, Samsung_Electro_Mechanics_CL05B104KO5NNNC:C0402, F.Cu at (10.0, -48.0)
- added D9: , STMicroelectronics_USBLC6_2SC6:SOT-23-6_L2.9-W1.6-P0.95-LS2.8-BL, F.Cu at (0.00, -5.75)
- added F3: , BHFUSE_BSMD0805_050_15V:F0805, F.Cu at (-4.00, -5.50)
- added J1: , HANRUN_HR911105A:RJ45-TH_HR911105A, F.Cu at (0.00, 0.00)
- added R56: 240Ω ±1%, YAGEO_RC0402FR_07240RL:R0402, F.Cu at (10.0, -84.0)
- added R57: 10kΩ ±1%, UNI_ROYAL_0603WAF1002T5E:R0603, F.Cu at (-2.25, -5.75)
- added R58: 10kΩ ±1%, UNI_ROYAL_0603WAF1002T5E:R0603, F.Cu at (3.50, -5.75)
- added R59: 10kΩ ±1%, UNI_ROYAL_0402WGF1002TCE:R0402, F.Cu at (20.0, -5.00)
- added R60: 4.7kΩ ±1%, UNI_ROYAL_0402WGF4701TCE:R0402, F.Cu at (20.0, -10.0)
- added R61: 4.7kΩ ±1%, UNI_ROYAL_0402WGF4701TCE:R0402, F.Cu at (20.0, -15.0)
- added R62: 1MΩ ±1%, UNI_ROYAL_0402WGF1004TCE:R0402, F.Cu at (10.0, -5.00)
- added R63: 330Ω ±1%, UNI_ROYAL_0402WGF3300TCE:R0402, F.Cu at (10.0, -10.0)
- added R64: 330Ω ±1%, UNI_ROYAL_0402WGF3300TCE:R0402, F.Cu at (10.0, -15.0)
- added R65: 75Ω ±1%, UNI_ROYAL_0402WGF750JTCE:R0402, F.Cu at (10.0, -20.0)
- added R66: 75Ω ±1%, UNI_ROYAL_0402WGF750JTCE:R0402, F.Cu at (10.0, -25.0)
- added U10: , Nanya_Tech_NT5CC128M16JR_EK:TFBGA-96_L13.0-W7.5-R16-C6-P0.80-TL, F.Cu at (0.00, 0.00)
- added U11: , NXP_Semicon_PCF8563T_5_518:SOIC-8_L5.0-W4.0-P1.27-LS6.0-BL, F.Cu at (0.00, 0.00)
- added USB3: , SHOU_HAN_TYPE_C_16PIN_2MD_073:USB-C-SMD_TYPE-C-6PIN-2MD-073, F.Cu at (0.00, 0.00)
- added X2: , Yangxing_Tech_X322524MOB4SI:CRYSTAL-SMD_4P-L3.2-W2.5-BL, F.Cu at (0.00, 0.00)
- added X3, X4: , Seiko_Epson_Q13FC13500004:FC-135R_L3.2-W1.5, F.Cu at (10.0, 0.00)
- R45: value 30kΩ ±1% -> 100kΩ ±1%; footprint UNI_ROYAL_0402WGF3002TCE:R0402 -> UNI_ROYAL_0402WGF1003TCE:R0402
- R46: value 20kΩ ±1% -> 100Ω ±1%; footprint UNI_ROYAL_0402WGF2002TCE:R0402 -> UNI_ROYAL_0402WGF1000TCE:R0402
- moved R45 258.8 mm to (30.0, 0.00)
- moved R46 258.8 mm to (30.0, -6.00)
Connections:
- net connector-cc[0]-4 renamed connector-cc[0]-4-1
- net connector-cc[1]-10 renamed connector-cc[1]-10-1
- net connector-power_vbus-hv-1 renamed connector-power_vbus-hv-2
- net connector-sbu[0]-9 renamed connector-sbu[0]-9-1
- net connector-sbu[1]-3 renamed connector-sbu[1]-3-1
- R45 pad 1: USB_OTG1_VBUS -> GPIO1_IO00
- R45 pad 2: cathode -> power_3v3-cathode
- R46 pad 1: usb_otg1_vbus_sense-line -> power_3v3-cathode
- U9 pad A7: A7 -> mpu-A7
- U9 pad D7: D7 -> mpu-D7
- U9 pad G16: UART4_RX_DATA -> SDA
- U9 pad G17: UART4_TX_DATA -> SCL
- U9 pad G2: DRAM_ADDR06 -> DDR_A6
- U9 pad H1: DRAM_SDBA1 -> BA1
- U9 pad H3: DRAM_ADDR13 -> DDR_A13
- U9 pad K13: usb_otg1_id-line -> GPIO1_IO00
- U9 pad K2: DRAM_SDBA2 -> BA2
- U9 pad K3: DRAM_ADDR11 -> DDR_A11
- U9 pad K4: DRAM_ADDR04 -> DDR_A4
- U9 pad L1: DRAM_ADDR05 -> DDR_A5
- U9 pad L4: DRAM_ADDR12 -> DDR_A12_nBC
- U9 pad L5: DRAM_ADDR00 -> DDR_A0
- U9 pad M1: DRAM_SDBA0 -> BA0
- U9 pad M16: GPIO1_IO04 -> nINT
- U9 pad M3: DRAM_SDCKE0 -> CKE
- U9 pad M4: DRAM_ADDR10 -> DDR_A10_AP
- U9 pad N1: DRAM_ODT0 -> ODT
- U9 pad P1: DRAM_SDCLK0_P -> CK
- U9 pad P3: DRAM_DATA13 -> A2
- U9 pad P5: DRAM_DATA12 -> A7
- U9 pad P6: DRAM_SDQS0_P -> DQSL
- U9 pad R1: DRAM_DATA15 -> A3
- U9 pad R2: DRAM_DATA14 -> B8
- U9 pad R4: DRAM_DATA11 -> C2
- U9 pad T1: DRAM_SDQS1_P -> DQSU
- U9 pad T15: USB_OTG1_DN_N -> usb_dp_dn-DATA_N
- U9 pad T3: DRAM_DQM1 -> DMU
- U9 pad T4: DRAM_DATA00 -> DQL0
- U9 pad T5: DRAM_DATA06 -> DQL6
- U9 pad T6: DRAM_DATA02 -> DQL2
- U9 pad T7: DRAM_DQM0 -> DML
- U9 pad T8: DRAM_DATA05 -> DQL5
- U9 pad U15: USB_OTG1_DP_P -> usb_dp_dn-DATA_P
- U9 pad U2: DRAM_DATA08 -> D7
- U9 pad U3: DRAM_DATA09 -> C3
- U9 pad U4: DRAM_DATA07 -> DQL7
- U9 pad U5: DRAM_DATA10 -> C8
- U9 pad U6: DRAM_DATA01 -> DQL1
- U9 pad U7: DRAM_DATA03 -> DQL3
- U9 pad U8: DRAM_DATA04 -> DQL4
Routing:
- net 0: track 103.6 -> 114.4 mm, vias 30 -> 33
- net cathode: track 0.00 -> 10.6 mm
- net connector-cc[1]-10: track 0.00 -> 10.0 mm, vias 0 -> 3
- net usb_dp_dn-DATA_N: track 0.00 -> 7.57 mm
- net usb_dp_dn-DATA_P: track 0.00 -> 6.68 mm
